File: PCB/Kicad5V/SD-10005v.kicad_sch (KiCad schematic)
At the start: 6 parts, among them CON1 SC3000-Edge, J1 Conn_01x20, J2 Conn_01x20, SW1 SW_Push

Commit message: Update PCB
-- Ground plane added to TOP & BOTTOM layer
-- Better routing for some tracks
-- Production files updated
-- JLCPCB DRU file added
Parts:
- D1: value Diode -> Diode
Changed lines of the file:
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@@
 			)
 		)
-		(property "Value" "Diode "
+		(property "Value" "Diode"
 			(at 128.27 58.42 0)
 			(effects
